File: PCBs/stepper_draft1.brd (EAGLE design)
At the start: 201.9 x 133 mm, 11 parts, among them J1 TBLH10V-500-04BK, J2 TBLH10V-500-04BK, J3 TBLH10V-500-04BK, J4 TBLH10V-500-04BK, U1 TMC2208_SILENTSTEPSTICK, U2 TMC2208_SILENTSTEPSTICK, U3 TMC2208_SILENTSTEPSTICK, U4 TMC2208_SILENTSTEPSTICK

Commit message: added modular neopixel data routing to schematic
added modular neopixel data routing to schematic
Parts:
- added JP1, JP2, JP3: (no value), jumper:JP2
- added LED1_IN, LED1_OUT, LED2_IN, LED2_OUT, LED3_IN, LED3_OUT, LED4_IN, LED4_OUT: TBLH10V-500-03BK, TBLH10V-500-03BK:CUI_TBLH10V-500-03BK
- added R1, R2, R3, R4: 1k, SparkFun-Resistors:AXIAL-0.3
Connections:
- new net LED_DATA_1: R1.P$1
- new net LED_DATA_2: R2.P$2
- new net LED_DATA_3: R3.P$1
- new net LED_DATA_4: R4.P$1
- new net N$17: LED1_IN.2_A, LED1_IN.2_B, R1.P$2
- new net N$18: JP1.3, LED1_OUT.2_A, LED1_OUT.2_B
- new net N$19: JP1.1, R2.P$1
- new net N$20: JP1.2, LED2_IN.2_A, LED2_IN.2_B
- new net N$21: JP2.3, LED2_OUT.2_A, LED2_OUT.2_B
- new net N$22: JP2.1, R3.P$2
- new net N$23: JP2.2, LED3_IN.2_A, LED3_IN.2_B
- new net N$24: JP3.1, R4.P$2
- new net N$25: JP3.3, LED3_OUT.2_A, LED3_OUT.2_B
- new net N$26: JP3.2, LED4_IN.2_A, LED4_IN.2_B
- new net VIN: LED1_IN.3_A, LED1_IN.3_B, LED1_OUT.3_A, LED1_OUT.3_B, LED2_IN.3_A, LED2_IN.3_B, LED2_OUT.3_A, LED2_OUT.3_B, LED3_IN.3_A, LED3_IN.3_B, LED3_OUT.3_A, LED3_OUT.3_B, LED4_IN.3_A, LED4_IN.3_B, LED4_OUT.3_A, LED4_OUT.3_B
- net GND: now also LED1_IN.1_A, LED1_IN.1_B, LED1_OUT.1_A, LED1_OUT.1_B, LED2_IN.1_A, LED2_IN.1_B, LED2_OUT.1_A, LED2_OUT.1_B, LED3_IN.1_A, LED3_IN.1_B, LED3_OUT.1_A, LED3_OUT.1_B, LED4_IN.1_A, LED4_IN.1_B, LED4_OUT.1_A, LED4_OUT.1_B
Other:
- board size 201.9 x 133 mm -> 201.9 x 202.9 mm

Commit message: minor PCB updates
minor PCB updates
Connections:
- removed net M5_DIR: B1.11
- removed net M5_STEP: B1.10
- removed net M6_DIR: B1.13
- removed net M6_STEP: B1.12
- new net N$27: B1.22
- new net N$28: B1.24
- new net N$29: B1.26
- new net N$30: B1.28
- new net N$31: B1.30
- new net N$32: B1.32
- new net N$33: B1.34
- new net N$34: B1.36
- new net N$35: B1.38
- new net N$36: B1.40
- new net N$37: B1.42
- new net N$38: B1.44
- new net N$39: B1.46
- new net N$40: B1.48
- new net N$41: B1.23
- new net N$42: B1.25
- new net N$43: B1.27
- new net N$44: B1.29
- new net N$45: B1.31
- new net N$46: B1.33
- new net N$47: B1.35
- new net N$48: B1.37
- new net N$49: B1.39
- new net N$50: B1.41
- new net N$51: B1.43
- new net N$52: B1.45
- new net N$53: B1.47
- new net N$54: B1.49
- new net N$55: B1.2
- new net N$56: B1.3
- new net N$57: B1.4
- new net N$58: B1.5
- new net N$59: B1.6
- new net N$60: B1.7
- net M1_DIR: no longer B1.3
- net M1_STEP: no longer B1.2
- net M2_DIR: no longer B1.5
- net M2_STEP: no longer B1.4
- net M3_DIR: no longer B1.7
- net M3_STEP: no longer B1.6
- net M4_DIR: no longer B1.9
- net M4_STEP: no longer B1.8
Changed lines of the file:
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@@
 </signal>
 <signal name="M1_STEP">
-<contactref element="B1" pad="2"/>
 <contactref element="U1" pad="JP1_2"/>
-<wire x1="60.96" y1="53.34" x2="27.94" y2="101.6" width="0" layer="19" extent="1-1"/>
 </signal>
 <signal name="M1_DIR">
-<contactref element="B1" pad="3"/>
 <contactref element="U1" pad="JP1_1"/>
-<wire x1="58.42" y1="53.34" x2="30.48" y2="101.6" width="0" layer="19" extent="1-1"/>
 </signal>
 <signal name="M2_STEP">
-<contactref element="B1" pad="4"/>
 <contactref element="U2" pad="JP1_2"/>
-<wire x1="55.88" y1="53.34" x2="57.15" y2="101.6" width="0" layer="19" extent="1-1"/>
 </signal>
 <signal name="M2_DIR">
-<contactref element="B1" pad="5"/>
 <contactref element="U2" pad="JP1_1"/>
-<wire x1="53.34" y1="53.34" x2="59.69" y2="101.6" width="0" layer="19" extent="1-1"/>
 </signal>
 <signal name="M3_STEP">
-<contactref element="B1" pad="6"/>
 <contactref element="U3" pad="JP1_2"/>
-<wire x1="50.8" y1="53.34" x2="86.36" y2="101.6" width="0" layer="19" extent="1-1"/>
 </signal>
 <signal name="M3_DIR">
-<contactref element="B1" pad="7"/>
 <contactref element="U3" pad="JP1_1"/>
-<wire x1="48.26" y1="53.34" x2="88.9" y2="101.6" width="0" layer="19" extent="1-1"/>
 </signal>
 <signal name="M4_STEP">
-<contactref element="B1" pad="8"/>
 <contactref element="U4" pad="JP1_2"/>
-<wire x1="44.45" y1="53.34" x2="115.57" y2="101.6" width="0" layer="19" extent="1-1"/>
-</signal>
-<signal name="M5_STEP">
-<contactref element="B1" pad="10"/>
-</signal>
-<signal name="M6_STEP">
-<contactref element="B1" pad="12"/>
 </signal>
 <signal name="M4_DIR">
-<contactref element="B1" pad="9"/>
 <contactref element="U4" pad="JP1_1"/>
-<wire x1="41.91" y1="53.34" x2="118.11" y2="101.6" width="0" layer="19" extent="1-1"/>
-</signal>
-<signal name="M5_DIR">
-<contactref element="B1" pad="11"/>
-</signal>
-<signal name="M6_DIR">
-<contactref element="B1" pad="13"/>
 </signal>
 <signal name="MS1">
@@
 <contactref element="R4" pad="P$1"/>
 </signal>
+<signal name="N$27">
+<contactref element="B1" pad="22"/>
+</signal>
+<signal name="N$28">
+<contactref element="B1" pad="24"/>
+</signal>
+<signal name="N$29">
+<contactref element="B1" pad="26"/>
+</signal>
+<signal name="N$30">
+<contactref element="B1" pad="28"/>
+</signal>
+<signal name="N$31">
+<contactref element="B1" pad="30"/>
+</signal>
+<signal name="N$32">
+<contactref element="B1" pad="32"/>
+</signal>
+<signal name="N$33">
+<contactref element="B1" pad="34"/>
+</signal>
+<signal name="N$34">
+<contactref element="B1" pad="36"/>
+</signal>
+<signal name="N$35">
+<contactref element="B1" pad="38"/>
+</signal>
+<signal name="N$36">
+<contactref element="B1" pad="40"/>
+</signal>
+<signal name="N$37">
+<contactref element="B1" pad="42"/>
+</signal>
+<signal name="N$38">
+<contactref element="B1" pad="44"/>
+</signal>
+<signal name="N$39">
+<contactref element="B1" pad="46"/>
+</signal>
+<signal name="N$40">
+<contactref element="B1" pad="48"/>
+</signal>
+<signal name="N$41">
+<contactref element="B1" pad="23"/>
+</signal>
+<signal name="N$42">
+<contactref element="B1" pad="25"/>
+</signal>
+<signal name="N$43">
+<contactref element="B1" pad="27"/>
+</signal>
+<signal name="N$44">
+<contactref element="B1" pad="29"/>
+</signal>
+<signal name="N$45">
+<contactref element="B1" pad="31"/>
+</signal>
+<signal name="N$46">
+<contactref element="B1" pad="33"/>
+</signal>
+<signal name="N$47">
+<contactref element="B1" pad="35"/>
+</signal>
+<signal name="N$48">
+<contactref element="B1" pad="37"/>
+</signal>
+<signal name="N$49">
+<contactref element="B1" pad="39"/>
+</signal>
+<signal name="N$50">
+<contactref element="B1" pad="41"/>
+</signal>
+<signal name="N$51">
+<contactref element="B1" pad="43"/>
+</signal>
+<signal name="N$52">
+<contactref element="B1" pad="45"/>
+</signal>
+<signal name="N$53">
+<contactref element="B1" pad="47"/>
+</signal>
+<signal name="N$54">
+<contactref element="B1" pad="49"/>
+</signal>
+<signal name="N$55">
+<contactref element="B1" pad="2"/>
+</signal>
+<signal name="N$56">
+<contactref element="B1" pad="3"/>
+</signal>
+<signal name="N$57">
+<contactref element="B1" pad="4"/>
+</signal>
+<signal name="N$58">
+<contactref element="B1" pad="5"/>
+</signal>
+<signal name="N$59">
+<contactref element="B1" pad="6"/>
+</signal>
+<signal name="N$60">
+<contactref element="B1" pad="7"/>
+</signal>
 </signals>

Commit message: added all 16 stepper drive packages to pcb
added all 16 stepper drive packages to pcb
Parts:
- added FRAME1: FRAME-LETTERNO_PACKAGE, SparkFun-Aesthetics:DUMMY
- added J10, J11, J12, J13, J14, J15, J16, J5, J6, J7, J8, J9: TBLH10V-500-04BK, TBLH10V-500-04BK:CUI_TBLH10V-500-04BK
- added U10, U11, U12, U13, U14, U15, U16, U5, U6, U7, U8, U9: TMC2208_SILENTSTEPSTICK, TMC2208_SILENTSTEPSTICK:MODULE_TMC2208_SILENTSTEPSTICK
- moved LED2_IN 322.8 mm to (185.4, 212.1), turned to 180 degrees
- moved R2 301.7 mm to (181.6, 196.8)
- moved JP1 300.7 mm to (180.3, 203.2)
- moved R3 293.8 mm to (25.4, 201.9), turned to 270 degrees
- moved LED1_OUT 290.7 mm to (191.8, 196.8), turned to 90 degrees
- moved JP2 282.9 mm to (17.8, 200.7), turned to 90 degrees
- moved LED3_IN 282.5 mm to (8.89, 205.7), turned to 270 degrees
- moved LED2_OUT 275.0 mm to (24.1, 212.1), turned to 180 degrees
- moved LED4_OUT 237.8 mm to (176.5, 10.2)
- moved LED1_IN 193.1 mm to (191.8, 16.5), turned to 90 degrees
- moved R1 190.0 mm to (182.9, 21.6)
- moved R4 169.6 mm to (22.9, 22.9)
- moved JP3 156.2 mm to (21.6, 17.8), turned to 180 degrees
- moved LED4_IN 126.7 mm to (16.5, 10.2)
- moved LED3_OUT 125.1 mm to (10.2, 25.4), turned to 270 degrees
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Connections:
- new net M10_DIR: B1.41, U10.JP1_1
- new net M10_STEP: B1.40, U10.JP1_2
- new net M11_DIR: B1.43, U11.JP1_1
- new net M11_STEP: B1.42, U11.JP1_2
- new net M12_DIR: B1.45, U12.JP1_1
- new net M12_STEP: B1.44, U12.JP1_2
- new net M13_DIR: B1.47, U13.JP1_1
- new net M13_STEP: B1.46, U13.JP1_2
- new net M14_DIR: B1.49, U14.JP1_1
- new net M14_STEP: B1.48, U14.JP1_2
- new net M15_DIR: B1.15, U15.JP1_1
- new net M15_STEP: B1.14, U15.JP1_2
- new net M16_DIR: B1.17, U16.JP1_1
- new net M16_STEP: B1.16, U16.JP1_2
- new net M5_DIR: B1.31, U5.JP1_1
- new net M5_STEP: B1.30, U5.JP1_2
- new net M6_DIR: B1.33, U6.JP1_1
- new net M6_STEP: B1.32, U6.JP1_2
- new net M7_DIR: B1.35, U7.JP1_1
- new net M7_STEP: B1.34, U7.JP1_2
- new net M8_DIR: B1.37, U8.JP1_1
- new net M8_STEP: B1.36, U8.JP1_2
- new net M9_DIR: B1.39, U9.JP1_1
- new net M9_STEP: B1.38, U9.JP1_2
- new net N$61: J14.4_A, J14.4_B, U14.JP2_6
- new net N$62: J14.3_A, J14.3_B, U14.JP2_5
- new net N$63: J14.2_A, J14.2_B, U14.JP2_4
- new net N$64: J14.1_A, J14.1_B, U14.JP2_3
- new net N$65: B1.9
- new net N$66: B1.8
- new net N$67: J9.4_A, J9.4_B, U9.JP2_6
- new net N$68: J9.3_A, J9.3_B, U9.JP2_5
- new net N$69: J9.2_A, J9.2_B, U9.JP2_4
- new net N$70: J9.1_A, J9.1_B, U9.JP2_3
- new net N$71: J10.4_A, J10.4_B, U10.JP2_6
- new net N$72: J10.3_A, J10.3_B, U10.JP2_5
- new net N$73: J10.2_A, J10.2_B, U10.JP2_4
- new net N$74: J10.1_A, J10.1_B, U10.JP2_3
- new net N$75: J11.4_A, J11.4_B, U11.JP2_6
- new net N$76: J11.3_A, J11.3_B, U11.JP2_5
- new net N$77: J11.2_A, J11.2_B, U11.JP2_4
- new net N$78: J11.1_A, J11.1_B, U11.JP2_3
- new net N$79: J12.4_A, J12.4_B, U12.JP2_6
- new net N$80: J12.3_A, J12.3_B, U12.JP2_5
- new net N$81: J12.2_A, J12.2_B, U12.JP2_4
- new net N$82: J12.1_A, J12.1_B, U12.JP2_3
- new net N$91: J15.4_A, J15.4_B, U15.JP2_6
- new net N$92: J15.3_A, J15.3_B, U15.JP2_5
- new net N$93: J15.2_A, J15.2_B, U15.JP2_4
- new net N$94: J15.1_A, J15.1_B, U15.JP2_3
- new net N$95: J16.4_A, J16.4_B, U16.JP2_6
- new net N$96: J16.3_A, J16.3_B, U16.JP2_5
- new net N$97: J16.2_A, J16.2_B, U16.JP2_4
- new net N$98: J16.1_A, J16.1_B, U16.JP2_3
- net 5V: now also U10.JP2_7, U11.JP2_7, U12.JP2_7, U13.JP2_7, U14.JP2_7, U15.JP2_7, U16.JP2_7, U5.JP2_7, U6.JP2_7, U7.JP2_7, U8.JP2_7, U9.JP2_7
- net GND: now also U10.JP2_2, U10.JP2_8, U11.JP2_2, U11.JP2_8, U12.JP2_2, U12.JP2_8, U13.JP2_2, U13.JP2_8, U14.JP2_2, U14.JP2_8, U15.JP2_2, U15.JP2_8, U16.JP2_2, U16.JP2_8, U5.JP2_2, U5.JP2_8, U6.JP2_2, U6.JP2_8, U7.JP2_2, U7.JP2_8, U8.JP2_2, U8.JP2_8, U9.JP2_2, U9.JP2_8
- net LED_DATA_1: now also B1.10
- net LED_DATA_2: now also B1.11
- net LED_DATA_3: now also B1.12
- net LED_DATA_4: now also B1.13
- net M1_DIR: now also B1.23
- net M1_STEP: now also B1.22
- net M2_DIR: now also B1.25
- net M2_STEP: now also B1.24
- net M3_DIR: now also B1.27
- net M3_STEP: now also B1.26
- net M4_DIR: now also B1.29
- net M4_STEP: now also B1.28
- net MS1: now also U10.JP1_7, U11.JP1_7, U12.JP1_7, U13.JP1_7, U14.JP1_7, U15.JP1_7, U16.JP1_7, U5.JP1_7, U6.JP1_7, U7.JP1_7, U8.JP1_7, U9.JP1_7
- net MS2: now also U10.JP1_6, U11.JP1_6, U12.JP1_6, U13.JP1_6, U14.JP1_6, U15.JP1_6, U16.JP1_6, U5.JP1_6, U6.JP1_6, U7.JP1_6, U8.JP1_6, U9.JP1_6
- net N$27: now also B1.A15; no longer B1.22
- net N$28: now also B1.A13; no longer B1.24
- net N$29: now also B1.A11; no longer B1.26
- net N$30: now also B1.A9; no longer B1.28
- net N$31: now also B1.A14; no longer B1.30
- net N$32: now also B1.A12; no longer B1.32
- net N$33: now also B1.A10; no longer B1.34
- net N$34: now also B1.A8; no longer B1.36
- net N$35: now also J5.4_A, J5.4_B, U5.JP2_6; no longer B1.38
- net N$36: now also J5.3_A, J5.3_B, U5.JP2_5; no longer B1.40
- net N$37: now also J5.2_A, J5.2_B, U5.JP2_4; no longer B1.42
- net N$38: now also J5.1_A, J5.1_B, U5.JP2_3; no longer B1.44
- net N$39: now also J6.4_A, J6.4_B, U6.JP2_6; no longer B1.46
- net N$40: now also J6.3_A, J6.3_B, U6.JP2_5; no longer B1.48
- net N$41: now also J6.2_A, J6.2_B, U6.JP2_4; no longer B1.23
- net N$42: now also J6.1_A, J6.1_B, U6.JP2_3; no longer B1.25
- net N$43: now also J7.4_A, J7.4_B, U7.JP2_6; no longer B1.27
- net N$44: now also J7.3_A, J7.3_B, U7.JP2_5; no longer B1.29
- net N$45: now also J7.2_A, J7.2_B, U7.JP2_4; no longer B1.31
- net N$46: now also J7.1_A, J7.1_B, U7.JP2_3; no longer B1.33
- net N$47: now also J8.4_A, J8.4_B, U8.JP2_6; no longer B1.35
- net N$48: now also J8.3_A, J8.3_B, U8.JP2_5; no longer B1.37
- net N$49: now also J8.2_A, J8.2_B, U8.JP2_4; no longer B1.39
- net N$50: now also J8.1_A, J8.1_B, U8.JP2_3; no longer B1.41
- net N$51: now also J13.4_A, J13.4_B, U13.JP2_6; no longer B1.43
- net N$52: now also J13.3_A, J13.3_B, U13.JP2_5; no longer B1.45
- net N$53: now also J13.2_A, J13.2_B, U13.JP2_4; no longer B1.47
- net N$54: now also J13.1_A, J13.1_B, U13.JP2_3; no longer B1.49
- net VCC: now also U10.JP2_1, U11.JP2_1, U12.JP2_1, U13.JP2_1, U14.JP2_1, U15.JP2_1, U16.JP2_1, U5.JP2_1, U6.JP2_1, U7.JP2_1, U8.JP2_1, U9.JP2_1
Routing:
- net VCC: track 0.00 -> 193.8 mm
- net VIN: track 0.00 -> 44.0 mm
- net N$23: track 0.00 -> 14.4 mm
- net N$82: track 0.00 -> 13.0 mm
- net N$78: track 0.00 -> 13.0 mm
- net N$50: track 0.00 -> 13.0 mm
- net N$46: track 0.00 -> 13.0 mm
- net N$70: track 0.00 -> 13.0 mm
- net N$38: track 0.00 -> 13.0 mm
- net N$74: track 0.00 -> 13.0 mm
- net N$42: track 0.00 -> 13.0 mm
- net N$98: track 0.00 -> 13.0 mm
- net N$94: track 0.00 -> 13.0 mm
- net N$8: track 0.00 -> 13.0 mm
- net N$54: track 0.00 -> 13.0 mm
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Other:
- board size 201.9 x 202.9 mm -> 201.9 x 221.9 mm

Commit message: started top layer routing
started top layer routing
Parts:
- moved SJ2 161.3 mm to (171.4, 101.6), turned to 270 degrees
- moved SJ1 155.8 mm to (167.6, 101.6), turned to 270 degrees
- moved B1 9.25 mm to (61.0, 58.4)
Routing:
- net MS2: track 0.00 -> 661.0 mm
- net VCC: track 193.8 -> 518.4 mm
- net VIN: track 44.0 -> 280.4 mm
- net MS1: track 0.00 -> 193.8 mm
- net LED_DATA_3: track 0.00 -> 131.3 mm
- net LED_DATA_4: track 0.00 -> 71.6 mm
- net N$25: track 5.50 -> 15.5 mm
- net N$18: track 5.50 -> 14.9 mm
- net N$21: track 5.50 -> 14.9 mm
- net N$20: track 5.50 -> 14.4 mm
- net N$26: track 5.50 -> 13.2 mm
- net N$22: track 0.00 -> 7.62 mm
- net N$24: track 0.00 -> 6.88 mm
- net N$19: track 0.00 -> 6.35 mm
- net N$17: track 5.50 -> 10.6 mm
- added copper zone on layer 1, net GND
Other:
- board size 201.9 x 221.9 mm -> 201.9 x 225.7 mm
