File: PCBs/stepper_draft1.sch (EAGLE design)
At the start: 11 parts, among them J1 TBLH10V-500-04BK, J2 TBLH10V-500-04BK, J3 TBLH10V-500-04BK, J4 TBLH10V-500-04BK, U1 TMC2208_SILENTSTEPSTICK, U2 TMC2208_SILENTSTEPSTICK, U3 TMC2208_SILENTSTEPSTICK, U4 TMC2208_SILENTSTEPSTICK

Commit message: added modular neopixel data routing to schematic
added modular neopixel data routing to schematic
Parts:
- added JP1, JP2, JP3: (no value), jumper:JP2E
- added LED1_IN, LED1_OUT, LED2_IN, LED2_OUT, LED3_IN, LED3_OUT, LED4_IN, LED4_OUT: TBLH10V-500-03BK, TBLH10V-500-03BK:TBLH10V-500-03BK
- added R1, R2, R3, R4: 1k, SparkFun-Resistors:1KOHM-HORIZ-1/4W-5%
Connections:
- new net LED_DATA_1: R1.1
- new net LED_DATA_2: R2.2
- new net LED_DATA_3: R3.1
- new net LED_DATA_4: R4.1
- new net N$17: LED1_IN.2, R1.2
- new net N$18: JP1.3, LED1_OUT.2
- new net N$19: JP1.1, R2.1
- new net N$20: JP1.2, LED2_IN.2
- new net N$21: JP2.3, LED2_OUT.2
- new net N$22: JP2.1, R3.2
- new net N$23: JP2.2, LED3_IN.2
- new net N$24: JP3.1, R4.2
- new net N$25: JP3.3, LED3_OUT.2
- new net N$26: JP3.2, LED4_IN.2
- new net VIN: LED1_IN.3, LED1_OUT.3, LED2_IN.3, LED2_OUT.3, LED3_IN.3, LED3_OUT.3, LED4_IN.3, LED4_OUT.3
- net GND: now also LED1_IN.1, LED1_OUT.1, LED2_IN.1, LED2_OUT.1, LED3_IN.1, LED3_OUT.1, LED4_IN.1, LED4_OUT.1

Commit message: minor PCB updates
minor PCB updates
Connections:
- removed net M5_DIR: B1.11
- removed net M5_STEP: B1.10
- removed net M6_DIR: B1.13
- removed net M6_STEP: B1.12
- new net N$27: B1.22
- new net N$28: B1.24
- new net N$29: B1.26
- new net N$30: B1.28
- new net N$31: B1.30
- new net N$32: B1.32
- new net N$33: B1.34
- new net N$34: B1.36
- new net N$35: B1.38
- new net N$36: B1.40
- new net N$37: B1.42
- new net N$38: B1.44
- new net N$39: B1.46
- new net N$40: B1.48
- new net N$41: B1.23
- new net N$42: B1.25
- new net N$43: B1.27
- new net N$44: B1.29
- new net N$45: B1.31
- new net N$46: B1.33
- new net N$47: B1.35
- new net N$48: B1.37
- new net N$49: B1.39
- new net N$50: B1.41
- new net N$51: B1.43
- new net N$52: B1.45
- new net N$53: B1.47
- new net N$54: B1.49
- new net N$55: B1.2
- new net N$56: B1.3
- new net N$57: B1.4
- new net N$58: B1.5
- new net N$59: B1.6
- new net N$60: B1.7
- net M1_DIR: no longer B1.3
- net M1_STEP: no longer B1.2
- net M2_DIR: no longer B1.5
- net M2_STEP: no longer B1.4
- net M3_DIR: no longer B1.7
- net M3_STEP: no longer B1.6
- net M4_DIR: no longer B1.9
- net M4_STEP: no longer B1.8

Commit message: added all 16 stepper drive packages to pcb
added all 16 stepper drive packages to pcb
Parts:
- added FRAME1: FRAME-LETTERNO_PACKAGE, SparkFun-Aesthetics:FRAME-LETTERNO_PACKAGE
- added J10, J11, J12, J13, J14, J15, J16, J5, J6, J7, J8, J9: TBLH10V-500-04BK, TBLH10V-500-04BK:TBLH10V-500-04BK
- added U10, U11, U12, U13, U14, U15, U16, U5, U6, U7, U8, U9: TMC2208_SILENTSTEPSTICK, TMC2208_SILENTSTEPSTICK:TMC2208_SILENTSTEPSTICK
Connections:
- new net M10_DIR: B1.41, U10.DIR
- new net M10_STEP: B1.40, U10.STEP
- new net M11_DIR: B1.43, U11.DIR
- new net M11_STEP: B1.42, U11.STEP
- new net M12_DIR: B1.45, U12.DIR
- new net M12_STEP: B1.44, U12.STEP
- new net M13_DIR: B1.47, U13.DIR
- new net M13_STEP: B1.46, U13.STEP
- new net M14_DIR: B1.49, U14.DIR
- new net M14_STEP: B1.48, U14.STEP
- new net M15_DIR: B1.15(RX3), U15.DIR
- new net M15_STEP: B1.14(TX3), U15.STEP
- new net M16_DIR: B1.17(RX2), U16.DIR
- new net M16_STEP: B1.16(TX2), U16.STEP
- new net M5_DIR: B1.31, U5.DIR
- new net M5_STEP: B1.30, U5.STEP
- new net M6_DIR: B1.33, U6.DIR
- new net M6_STEP: B1.32, U6.STEP
- new net M7_DIR: B1.35, U7.DIR
- new net M7_STEP: B1.34, U7.STEP
- new net M8_DIR: B1.37, U8.DIR
- new net M8_STEP: B1.36, U8.STEP
- new net M9_DIR: B1.39, U9.DIR
- new net M9_STEP: B1.38, U9.STEP
- new net N$61: J14.4, U14.OB2
- new net N$62: J14.3, U14.OB1
- new net N$63: J14.2, U14.OA1
- new net N$64: J14.1, U14.OA2
- new net N$65: B1.9
- new net N$66: B1.8
- new net N$67: J9.4, U9.OB2
- new net N$68: J9.3, U9.OB1
- new net N$69: J9.2, U9.OA1
- new net N$70: J9.1, U9.OA2
- new net N$71: J10.4, U10.OB2
- new net N$72: J10.3, U10.OB1
- new net N$73: J10.2, U10.OA1
- new net N$74: J10.1, U10.OA2
- new net N$75: J11.4, U11.OB2
- new net N$76: J11.3, U11.OB1
- new net N$77: J11.2, U11.OA1
- new net N$78: J11.1, U11.OA2
- new net N$79: J12.4, U12.OB2
- new net N$80: J12.3, U12.OB1
- new net N$81: J12.2, U12.OA1
- new net N$82: J12.1, U12.OA2
- new net N$91: J15.4, U15.OB2
- new net N$92: J15.3, U15.OB1
- new net N$93: J15.2, U15.OA1
- new net N$94: J15.1, U15.OA2
- new net N$95: J16.4, U16.OB2
- new net N$96: J16.3, U16.OB1
- new net N$97: J16.2, U16.OA1
- new net N$98: J16.1, U16.OA2
- net 5V: now also U10.VIO, U11.VIO, U12.VIO, U13.VIO, U14.VIO, U15.VIO, U16.VIO, U5.VIO, U6.VIO, U7.VIO, U8.VIO, U9.VIO
- net GND: now also U10.GND, U11.GND, U12.GND, U13.GND, U14.GND, U15.GND, U16.GND, U5.GND, U6.GND, U7.GND, U8.GND, U9.GND
- net LED_DATA_1: now also B1.10
- net LED_DATA_2: now also B1.11
- net LED_DATA_3: now also B1.12
- net LED_DATA_4: now also B1.13
- net M1_DIR: now also B1.23
- net M1_STEP: now also B1.22
- net M2_DIR: now also B1.25
- net M2_STEP: now also B1.24
- net M3_DIR: now also B1.27
- net M3_STEP: now also B1.26
- net M4_DIR: now also B1.29
- net M4_STEP: now also B1.28
- net MS1: now also U10.MS1, U11.MS1, U12.MS1, U13.MS1, U14.MS1, U15.MS1, U16.MS1, U5.MS1, U6.MS1, U7.MS1, U8.MS1, U9.MS1
- net MS2: now also U10.MS2, U11.MS2, U12.MS2, U13.MS2, U14.MS2, U15.MS2, U16.MS2, U5.MS2, U6.MS2, U7.MS2, U8.MS2, U9.MS2
- net N$27: now also B1.A15; no longer B1.22
- net N$28: now also B1.A13; no longer B1.24
- net N$29: now also B1.A11; no longer B1.26
- net N$30: now also B1.A9; no longer B1.28
- net N$31: now also B1.A14; no longer B1.30
- net N$32: now also B1.A12; no longer B1.32
- net N$33: now also B1.A10; no longer B1.34
- net N$34: now also B1.A8; no longer B1.36
- net N$35: now also J5.4, U5.OB2; no longer B1.38
- net N$36: now also J5.3, U5.OB1; no longer B1.40
- net N$37: now also J5.2, U5.OA1; no longer B1.42
- net N$38: now also J5.1, U5.OA2; no longer B1.44
- net N$39: now also J6.4, U6.OB2; no longer B1.46
- net N$40: now also J6.3, U6.OB1; no longer B1.48
- net N$41: now also J6.2, U6.OA1; no longer B1.23
- net N$42: now also J6.1, U6.OA2; no longer B1.25
- net N$43: now also J7.4, U7.OB2; no longer B1.27
- net N$44: now also J7.3, U7.OB1; no longer B1.29
- net N$45: now also J7.2, U7.OA1; no longer B1.31
- net N$46: now also J7.1, U7.OA2; no longer B1.33
- net N$47: now also J8.4, U8.OB2; no longer B1.35
- net N$48: now also J8.3, U8.OB1; no longer B1.37
- net N$49: now also J8.2, U8.OA1; no longer B1.39
- net N$50: now also J8.1, U8.OA2; no longer B1.41
- net N$51: now also J13.4, U13.OB2; no longer B1.43
- net N$52: now also J13.3, U13.OB1; no longer B1.45
- net N$53: now also J13.2, U13.OA1; no longer B1.47
- net N$54: now also J13.1, U13.OA2; no longer B1.49
- net VCC: now also U10.VM, U11.VM, U12.VM, U13.VM, U14.VM, U15.VM, U16.VM, U5.VM, U6.VM, U7.VM, U8.VM, U9.VM
Other:
- moved on the sheet: J1, J2, J3, J4, JP1, JP2, JP3, LED1_IN, LED1_OUT, LED2_IN, LED2_OUT, LED3_IN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
